File: ardiu-usb/ardiu-usb.kicad_pcb (KiCad board)
At the start: 2 copper layers, 39 parts, among them J1 ICSP, J2 Conn_01x06_Female, Q1 AO4838, Q2 AO4838, SW1 SW_Push, U1 ATmega328PB-A, U2 AP7375-33SA-7

Commit message: Ardiu USB progress
Parts:
- removed D4: LED, LED_THT:LED_D3.0mm
- removed H3, H4: MountingHole, MountingHole:MountingHole_3.2mm_M3
- removed J2: Conn_01x06_Female, Connector_PinSocket_2.54mm:PinSocket_1x06_P2.54mm_Vertical
- removed RN1: 100k, Resistor_SMD:R_Array_Concave_4x0603
- removed RN2, RN3, RN6: 10k, Resistor_SMD:R_Array_Concave_4x0603
- removed RN4, RN7: 220, Resistor_SMD:R_Array_Concave_4x0603
- removed RN5: 2200, Resistor_SMD:R_Array_Concave_4x0603
- removed TPX1, TPX2: x, TestPoint:TestPoint_Pad_D1.5mm
- removed U1: ATmega328PB-A, Package_QFP:TQFP-32_7x7mm_P0.8mm
- added ACCEL1: MPU6050, Sensor_BreakoutBoards:Breakout_MPU6050_Generic, F.Cu at (200.7, 90.2)
- added BARO1: BMP280, Sensor_BreakoutBoards:Breakout_BMP280_Generic, F.Cu at (177.8, 90.2)
- added C8: 1u, Capacitor_SMD:C_0805_2012Metric_Pad1.18x1.45mm_HandSolder, B.Cu at (212.1, 111.8)
- added J3: Micro_SD_Card_Det, Connector_Amphenol:Connector_Amphenol_MicroSD_PushPull, F.Cu at (193.0, 108.0)
- added J4: USB_C_Receptacle_USB2.0, Connector_USB:USB_C_Receptacle_GCT_USB4085, F.Cu at (218.0, 106.7)
- added R10: 10k, Resistor_SMD:R_0805_2012Metric_Pad1.20x1.40mm_HandSolder, B.Cu at (189.2, 95.5)
- added R11: 220, Resistor_SMD:R_0805_2012Metric_Pad1.20x1.40mm_HandSolder, B.Cu at (182.9, 96.5)
- added R12: 220, Resistor_SMD:R_0805_2012Metric_Pad1.20x1.40mm_HandSolder, B.Cu at (182.9, 94.0)
- added R13: 220, Resistor_SMD:R_0805_2012Metric_Pad1.20x1.40mm_HandSolder, B.Cu at (191.8, 100.6)
- added R14: 220, Resistor_SMD:R_0805_2012Metric_Pad1.20x1.40mm_HandSolder, B.Cu at (189.2, 100.6)
- added R15: 100k, Resistor_SMD:R_0805_2012Metric_Pad1.20x1.40mm_HandSolder, B.Cu at (166.4, 105.4)
- added R16: 10k, Resistor_SMD:R_0805_2012Metric_Pad1.20x1.40mm_HandSolder, B.Cu at (166.4, 101.6)
- added R17: 100k, Resistor_SMD:R_0805_2012Metric_Pad1.20x1.40mm_HandSolder, B.Cu at (174.0, 105.4)
- added R18: 10k, Resistor_SMD:R_0805_2012Metric_Pad1.20x1.40mm_HandSolder, B.Cu at (174.0, 101.6)
- added R19: 100k, Resistor_SMD:R_0805_2012Metric_Pad1.20x1.40mm_HandSolder, B.Cu at (176.5, 105.4)
- added R20: 10k, Resistor_SMD:R_0805_2012Metric_Pad1.20x1.40mm_HandSolder, B.Cu at (176.5, 101.6)
- added R21: 100k, Resistor_SMD:R_0805_2012Metric_Pad1.20x1.40mm_HandSolder, B.Cu at (184.2, 105.4)
- added R22: 10k, Resistor_SMD:R_0805_2012Metric_Pad1.20x1.40mm_HandSolder, B.Cu at (184.2, 101.3)
- added R23: 10k, Resistor_SMD:R_0805_2012Metric_Pad1.20x1.40mm_HandSolder, B.Cu at (171.2, 92.7)
- added R24: 10k, Resistor_SMD:R_0805_2012Metric_Pad1.20x1.40mm_HandSolder, B.Cu at (189.2, 111.8)
- added R25: 10k, Resistor_SMD:R_0805_2012Metric_Pad1.20x1.40mm_HandSolder, B.Cu at (193.0, 111.8)
- added R26: 220, Resistor_SMD:R_0805_2012Metric_Pad1.20x1.40mm_HandSolder, B.Cu at (214.6, 96.5)
- added R27: 220, Resistor_SMD:R_0805_2012Metric_Pad1.20x1.40mm_HandSolder, B.Cu at (214.6, 99.1)
- added R29: 10k, Resistor_SMD:R_0805_2012Metric_Pad1.20x1.40mm_HandSolder, B.Cu at (196.8, 111.8)
- added R3: 5.1k, Resistor_SMD:R_0805_2012Metric_Pad1.20x1.40mm_HandSolder, B.Cu at (222.2, 111.8)
- added R4: 22, Resistor_SMD:R_0805_2012Metric_Pad1.20x1.40mm_HandSolder, B.Cu at (210.8, 104.1)
- added R5: 5.1k, Resistor_SMD:R_0805_2012Metric_Pad1.20x1.40mm_HandSolder, B.Cu at (219.7, 111.8)
- added R6: 22, Resistor_SMD:R_0805_2012Metric_Pad1.20x1.40mm_HandSolder, B.Cu at (210.8, 101.6)
- added R7: 10k, Resistor_SMD:R_0805_2012Metric_Pad1.20x1.40mm_HandSolder, B.Cu at (177.8, 96.5)
- added R8: 10k, Resistor_SMD:R_0805_2012Metric_Pad1.20x1.40mm_HandSolder, B.Cu at (177.8, 94.0)
- added R9: 10k, Resistor_SMD:R_0805_2012Metric_Pad1.20x1.40mm_HandSolder, B.Cu at (191.8, 95.5)
- added U3: ATmega32U4-A, Package_QFP:TQFP-44_10x10mm_P0.8mm, B.Cu at (200.7, 102.9)
- added Y1: 8MHz, Crystal:Resonator_SMD_Murata_CSTxExxV-3Pin_3.0x1.1mm_HandSoldering, B.Cu at (201.9, 111.8)
- C1, C2, C3, C5, C6, C7, D1, Q1, Q2, R1, R2, U2: moved to B.Cu
- C4: value 0.1u -> 1u; moved to B.Cu
- moved BZ1 126.1 mm to (209.6, 106.7), turned to 90 degrees
- moved C3 110.5 mm to (204.5, 94.0), turned to 180 degrees
- moved H2 107.8 mm to (222.2, 95.2)
- moved C1 102.7 mm to (207.0, 111.8)
- moved D3 100.2 mm to (219.7, 102.9), turned to 90 degrees
- moved J1 99.9 mm to (208.3, 92.7), turned to 90 degrees
- moved D2 95.4 mm to (224.8, 102.9), turned to 90 degrees
- moved C4 91.9 mm to (212.1, 109.2), turned to 180 degrees
- moved JPYRO4 83.7 mm to (180.3, 109.2)
- moved U2 80.9 mm to (168.9, 96.5), turned to -90 degrees
- moved JPYRO3 79.3 mm to (175.3, 109.2)
- moved R1 78.5 mm to (166.6, 92.7)
- moved D1 77.4 mm to (161.3, 100.3), turned to 90 degrees
- moved C5 75.3 mm to (165.1, 96.5), turned to -90 degrees
- moved JPYRO2 74.9 mm to (170.2, 109.2)
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Connections:
- net Net-(C5-Pad1) renamed /VRIN
- C1 pad 1: Net-(C1-Pad1) -> +3V3
- C2 pad 1: +3V3 -> Net-(C2-Pad1)
- C4 pad 1: /DTR -> +5V
- C4 pad 2: /RST -> GND
- J1 pad 2: +5V -> +3V3
- J1 pad 3: /5SCK -> /SCK
- J1 pad 4: /5MOSI -> /MOSI
Routing:
- net /SENS4: track 0.00 -> 2.08 mm
- net /PYRO2: track 0.00 -> 2.03 mm
- net /PYRO4: track 0.00 -> 2.03 mm
- net /PYRO3: track 0.00 -> 2.03 mm
- net /PYRO1: track 0.00 -> 2.03 mm
- net /SENS3: track 0.00 -> 1.81 mm
- net /SENS2: track 0.00 -> 1.81 mm
- net /SENS1: track 0.00 -> 1.81 mm
- added copper zone on F.Cu, net +3V3
- added copper zone on B.Cu, net +BATT
- added copper zone on B.Cu, net /PYRO1
- added copper zone on B.Cu, net /PYRO2
- added copper zone on B.Cu, net /PYRO3
- added copper zone on B.Cu, net /PYRO4
- added copper zone on B.Cu, net GND
Other:
- board outline added: 76.2 x 25.4 mm
- rule pad_to_mask_clearance: 0 -> 0.0508
