File: ardiu-usb/ardiu-usb.kicad_sch (KiCad schematic)
At the start: 43 parts, among them J1 ICSP, J2 Conn_01x06_Female, J3 Micro_SD_Card_Det, Q1 AO4838, Q2 AO4838, SW1 SW_Push, U1 ATmega328PB-A, U2 AP7375-33SA-7

Commit message: Ardiu USB progress
Parts:
- removed D4: LED, LED_THT:LED_D3.0mm, symbol Device:LED
- removed H3, H4: MountingHole, MountingHole:MountingHole_3.2mm_M3, symbol Mechanical:MountingHole
- removed J2: Conn_01x06_Female, Connector_PinSocket_2.54mm:PinSocket_1x06_P2.54mm_Vertical, symbol Connector:Conn_01x06_Female
- removed RN1: 100k, Resistor_SMD:R_Array_Concave_4x0603, symbol Device:R_Pack04_Split
- removed RN2, RN3, RN6: 10k, Resistor_SMD:R_Array_Concave_4x0603, symbol Device:R_Pack04_Split
- removed RN4, RN7: 220, Resistor_SMD:R_Array_Concave_4x0603, symbol Device:R_Pack04_Split
- removed RN5: 2200, Resistor_SMD:R_Array_Concave_4x0603, symbol Device:R_Pack04_Split
- removed TPX1, TPX2: x, TestPoint:TestPoint_Pad_D1.5mm, symbol Connector:TestPoint
- removed U1: ATmega328PB-A, Package_QFP:TQFP-32_7x7mm_P0.8mm, symbol MCU_Microchip_ATmega:ATmega328PB-A
- added C8: 1u, Capacitor_SMD:C_0805_2012Metric_Pad1.18x1.45mm_HandSolder, symbol Device:C
- added J4: USB_C_Receptacle_USB2.0, Connector_USB:USB_C_Receptacle_GCT_USB4085, symbol Connector:USB_C_Receptacle_USB2.0
- added R10, R16, R18, R20, R22, R23, R24, R25, R29, R7, R8, R9: 10k, Resistor_SMD:R_0805_2012Metric_Pad1.20x1.40mm_HandSolder, symbol Device:R_US
- added R11, R12, R13, R14, R26, R27: 220, Resistor_SMD:R_0805_2012Metric_Pad1.20x1.40mm_HandSolder, symbol Device:R_US
- added R15, R17, R19, R21: 100k, Resistor_SMD:R_0805_2012Metric_Pad1.20x1.40mm_HandSolder, symbol Device:R_US
- added R3, R5: 5.1k, Resistor_SMD:R_0805_2012Metric_Pad1.20x1.40mm_HandSolder, symbol Device:R_US
- added R4, R6: 22, Resistor_SMD:R_0805_2012Metric_Pad1.20x1.40mm_HandSolder, symbol Device:R_US
- added Y1: 8MHz, Crystal:Resonator_SMD_Murata_CSTxExxV-3Pin_3.0x1.1mm_HandSoldering, symbol Device:Resonator
- C4: value 0.1u -> 1u
- J3: footprint Connector_Amphenol_Custom:Connector_Amphenol_MicroSD_PushPull -> Connector_Amphenol:Connector_Amphenol_MicroSD_PushPull
- gave numbers to parts that had none: 4
Connections:
- net 5MOSI is gone; now on net MOSI: J1.4 (Pin_4)
- net 5SCK is gone; now on net SCK: J1.3 (Pin_3)
- net DTR is gone; now on net +5V: C4.1
- net +3V3: now also J1.2 (Pin_2), R24.1, R25.1, R26.1, R29.1
- net +5V: now also U3.2 (UVCC), U3.7 (VBUS), J4.A4 (VBUS), J4.A9 (VBUS), J4.B4 (VBUS), J4.B9 (VBUS); no longer J1.2 (Pin_2)
- net BUZ: now also U3.32 (PC7)
- net CH1: now also U3.29 (PB5), R11.1, R7.1
- net CH2: now also U3.30 (PB6), R12.1, R8.1
- net CH3: now also U3.12 (PB7), R13.1, R9.1
- net CH4: now also U3.31 (PC6), R10.1, R14.1
- net CS_SD: now also U3.28 (PB4), R25.2
- net GND: now also C4.2, C8.2, J4.A1 (GND), J4.A12 (GND), J4.B1 (GND), J4.B12 (GND), J4.S1 (SHIELD), R10.2, R16.2, R18.2, R20.2, R22.2, R23.2, R3.2, R5.2, R7.2, R8.2, R9.2, Y1.2
- net INT: now also U3.1 (PE6)
- net LED: now also U3.8 (PB0), R27.1
- net MISO: now also U3.11 (PB3)
- net MOSI: now also U3.10 (PB2)
- net PYRO1: now also R15.1
- net PYRO2: now also R17.1
- net PYRO3: now also R19.1
- net PYRO4: now also R21.1
- net RLED: now also R27.2
- net RPWR: now also R26.2
- net RST: now also U3.13 (~{RESET}); no longer C4.2
- net RX: now also U3.20 (PD2)
- net SCK: now also U3.9 (PB1)
- net SCL: now also U3.18 (PD0)
- net SDA: now also U3.19 (PD1)
- net SENS1: now also U3.39 (PF4), R15.2, R16.1
- net SENS2: now also U3.38 (PF5), R17.2, R18.1
- net SENS3: now also U3.37 (PF6), R19.2, R20.1
- net SENS4: now also U3.36 (PF7), R21.2, R22.1
- net SENS_BATT: now also U3.41 (PF0), R23.1
- net TX: now also U3.21 (PD3)
- net at J3.8 (DAT1): now also R24.2
- net at Q2.4 (G): now also R14.2
- net at U3.16 (XTAL2): now also Y1.3
- net at U3.17 (XTAL1): now also Y1.1
- net at U3.3 (D-): now also R6.2
- net at U3.4 (D+): now also R4.2
- net at U3.6 (UCAP): now also C8.1
- net at Q1.2 (G): now also R11.2
- net at J3.1 (DAT2): now also R29.2
- net at Q2.2 (G): now also R13.2
- net at Q1.4 (G): now also R12.2
- new net: J4.A5 (CC1), R5.1
- new net: J4.A6 (D+), J4.B6 (D+), R4.1
- new net: J4.A7 (D-), J4.B7 (D-), R6.1
- new net: J4.B5 (CC2), R3.1
Other:
- note added: "Arduino Pin Assignments 0: RX 1: TX 2: SDA 3: SCL 4: 5: Ch4 out 6: 7: IMU interrupt 8: CS SD 9: Ch1 out 10: Ch2 out 11: Ch3 out 12: 13: Buzzer 14: MISO 15: SCK 16: MOSI 17: LED A0: Ch4 sense A1: Ch3 sense A2: Ch2 sense A3: Ch1 sense A4: A5: Battery sense"
- note removed: "Arduino Pin Assignments 0: RX 1: TX 2: Gyro Interrupt 3: Channel 1 Out 4: Channel 2 Out 5: Channel 3 Out 6: Channel 4 Out 7: Buzzer 8: LED 9: 10: SPI CS SD 11: SPI MOSI 12: SPI MISO 13: SPI SCK A0: Channel 1 sense A1: Channel 2 sense A2: Channel 3 sense A3: Channel 4 sense A4: SDA A5: SCL A6: Battery sense A7:"
- moved on the sheet: BZ1, C1, C2, C3, C5, C7, D1, D2, D3, JBAT1, JPYRO1, JPYRO2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
